File: PedalBoardStereoAmpTDA7297.kicad_pcb (KiCad board)
At the start: 2 copper layers, 49.5 x 27.9 mm, 17 parts, among them J1 OUT-L, J2 Conn_01x03_Male, J3 OUT-R, J5 PWR, U1 TDA7297

Commit message: update
Parts:
- J2: value Conn_01x03_Male -> 1/4
- J5: footprint Connector_PinHeader_2.54mm:PinHeader_1x02_P2.54mm_Vertical -> TerminalBlock:TerminalBlock_bornier-2_P5.08mm
- moved C3 15.4 mm to (99.8, 54.9), turned to 270 degrees
- moved R2 13.0 mm to (98.8, 48.8)
- moved R3 11.2 mm to (90.7, 63.5)
- moved C1 7.22 mm to (75.7, 53.8)
- moved J5 3.75 mm to (106.4, 58.2), turned to 90 degrees
- moved R1 2.97 mm to (96.3, 52.1)
- moved J2 2.30 mm to (74.2, 63.5)
- moved H2 2.29 mm to (63.5, 63.2)
- moved H4 2.29 mm to (108.0, 63.2)
- moved C2 1.80 mm to (93.0, 48.8)
- moved J3 0.51 mm to (108.2, 45.2)
Connections:
- J2 pad 1: Net-(J2-Pad1) -> Net-(J4-Pad1)
- J2 pad 2: Net-(J2-Pad2) -> Net-(J4-Pad2)
- R3 pad 1: Net-(J2-Pad1) -> Net-(R3-Pad1)
- R3 pad 4: Net-(J2-Pad2) -> Net-(R3-Pad4)
Routing:
- net Net-(R3-Pad4): track 0.00 -> 48.5 mm
- net Net-(R3-Pad1): track 0.00 -> 34.5 mm
- net Net-(C3-Pad1): track 18.7 -> 33.8 mm
- net Net-(J4-Pad1): track 0.00 -> 12.4 mm
- net Net-(J2-Pad2): track 18.1 -> 10.6 mm
- net Net-(C4-Pad2): track 27.0 -> 34.2 mm
- net Net-(J4-Pad2): track 0.00 -> 5.07 mm
- net Net-(J2-Pad1): track 5.84 -> 9.71 mm
- net Net-(C5-Pad2): track 23.0 -> 26.0 mm
Other:
- board size 49.5 x 27.9 mm -> 49.5 x 30.2 mm

Commit message: update design
Parts:
- moved J2 5.08 mm to (69.1, 63.5), turned to 90 degrees
- moved C3 0.90 mm to (98.9, 55.0)
- moved J1 0.51 mm to (64.0, 45.2)
- moved C2 0.13 mm to (93.0, 48.6)
- moved R2 0.13 mm to (98.8, 48.6)
- moved J5 0.13 mm to (106.4, 58.0)
Connections:
- net Net-(R3-Pad1) renamed LEFT
- net Net-(R3-Pad4) renamed RIGHT
- J2 pad 1: Net-(J4-Pad1) -> GND
- J2 pad 3: GND -> Net-(J4-Pad3)
Routing:
- net Net-(J4-Pad3): track 0.00 -> 13.0 mm
- net Net-(J4-Pad1): track 12.4 -> 0.00 mm
- net Net-(J2-Pad3): track 0.00 -> 10.4 mm
- net Net-(J2-Pad1): track 9.71 -> 0.00 mm
- net Net-(C5-Pad2): track 26.0 -> 21.9 mm
- net Net-(C4-Pad2): track 34.2 -> 37.8 mm
- net RIGHT: track 48.5 -> 46.7 mm
- net Net-(C3-Pad1): track 33.8 -> 32.7 mm
- net Net-(J2-Pad2): track 10.6 -> 11.2 mm
Other:
- board text added: "IN"
